Commit message: tested. aruco pose detected in gazebo is accurate. added tf in aruco, changed marker size, urdf

File: ur10_simulation/urdf/ur10.urdf.xacro (robot description, xacro)
@@ -346,17 +346,18 @@
       <parent link="mounting_plate" />
       <child link = "camera" />
-      <origin xyz=" 0.02 0.0 0.065" rpy="0.0 0.0 0.0" />
+      <origin xyz=" 0.00 0.0 0.065" rpy="-1.57 0.0 -1.57" />
    </joint>
   <link name="camera">
-    <collision>
-      <origin xyz="0 0 0" rpy="0 0 0"/>
+    <!--<collision>
+      <origin xyz="0 0 0" rpy="0 0 1.57"/>
       <geometry>
     <box size=" 0.05 0.15 0.05 "/>
       </geometry>
-    </collision>
+    </collision> -->
     <visual>
       <origin xyz="0 0 0" rpy="0 0 0"/>
       <geometry>
-    <box size=" 0.05 0.15 0.05 "/>
+    <box size=" 0.01 0.01 0.01 "/>
+<!--0.05 0.15 0.05 -->
       </geometry>
       <material name="red">
@@ -370,5 +371,13 @@
     </inertial>
   </link>
-<gazebo reference="camera">
+<joint name="camera_optical_joint" type="fixed">
+    <!-- satisfy both gazebo convention and aruco pkg convetion. looking from x axis and z axis respectively. -->
+    <origin xyz=" 0.0 0.0 0.065" rpy="0 0.0 0" />>
+    <parent link="mounting_plate"/>
+    <child link="camera_link_optical"/>
+  </joint>
+ <link name="camera_link_optical">
+  </link>
+<gazebo reference="camera_link_optical">
     <sensor type="camera" name="camera1">
       <update_rate>30.0</update_rate>
@@ -396,8 +405,8 @@
       <plugin name="camera_controller" filename="libgazebo_ros_camera.so">
         <alwaysOn>true</alwaysOn>
-        <updateRate>0.0</updateRate>
-        <cameraName>rrbot/camera1</cameraName>
+        <updateRate>60</updateRate>
+        <cameraName></cameraName>
         <imageTopicName>/image</imageTopicName>
-        <cameraInfoTopicName>camera_info</cameraInfoTopicName>
+        <cameraInfoTopicName>/camera_info</cameraInfoTopicName>
         <frameName>camera_link</frameName>
         <hackBaseline>0.07</hackBaseline>

Commit message: 4x4 fiducial tested to be accurate

File: ur10_simulation/urdf/ur10.urdf.xacro (robot description, xacro)
@@ -304,5 +304,5 @@
       <parent link="mounting_plate" />
       <child link = "fork_left" />
-      <origin xyz="0.131 -0.1 0.0" rpy="0.0 0.0 0.0" />
+      <origin xyz="0.16 -0.1 0.0" rpy="0.0 0.0 0.0" />
     </joint>
     <link name="fork_left">
@@ -312,10 +312,10 @@
         </material>
   <geometry>
-          <box size="0.25 0.01 0.01"/>
-        </geometry>
-      </visual>
-      <collision>
-        <geometry>
-          <box size="0.25 0.01 0.01"/>
+          <box size="0.3 0.01 0.01"/>
+        </geometry>
+      </visual>
+      <collision>
+        <geometry>
+          <box size="0.3 0.01 0.01"/>
         </geometry>
       </collision>
@@ -324,5 +324,5 @@
       <parent link="mounting_plate" />
       <child link = "fork_right" />
-      <origin xyz="0.131 0.1 0.0" rpy="0.0 0.0 0.0" />
+      <origin xyz="0.16 0.1 0.0" rpy="0.0 0.0 0.0" />
     </joint>
     <link name="fork_right">
@@ -332,10 +332,10 @@
         </material>
   <geometry>
-          <box size="0.25 0.01 0.01"/>
-        </geometry>
-      </visual>
-      <collision>
-        <geometry>
-          <box size="0.25 0.01 0.01"/>
+          <box size="0.3 0.01 0.01"/>
+        </geometry>
+      </visual>
+      <collision>
+        <geometry>
+          <box size="0.3 0.01 0.01"/>
         </geometry>
       </collision>
@@ -383,8 +383,8 @@
       <update_rate>30.0</update_rate>
       <camera name="camera_head">
-        <horizontal_fov>2.094</horizontal_fov>
+        <horizontal_fov>1.57</horizontal_fov>
         <image>
-          <width>640</width>
-          <height>480</height>
+          <width>3840</width>
+          <height>1080</height>
           <!--<format>R8G8B8</format> -->
           <format>R8G8B8</format>
@@ -405,5 +405,5 @@
       <plugin name="camera_controller" filename="libgazebo_ros_camera.so">
         <alwaysOn>true</alwaysOn>
-        <updateRate>60</updateRate>
+        <updateRate>30</updateRate>
         <cameraName></cameraName>
         <imageTopicName>/image</imageTopicName>

Commit message: ee link

File: ur10_simulation/urdf/ur10.urdf.xacro (robot description, xacro)
@@ -1,8 +1,4 @@
 <?xml version="1.0"?>
 <robot xmlns:xacro="http://wiki.ros.org/xacro">
-<!--
-  Author: Kelsey Hawkins
-  Contributers: Jimmy Da Silva, Ajit Krisshna N L, Muhammad Asif Rana
--->
   <xacro:include filename="$(find ur_description)/urdf/ur.transmission.xacro" />
   <xacro:include filename="$(find ur_description)/urdf/ur.gazebo.xacro" />
@@ -277,147 +273,25 @@
       </collision>
     </link>
-    <xacro:ur_arm_transmission prefix="${prefix}" hw_interface="${transmission_hw_interface}" />
-    <xacro:ur_arm_gazebo prefix="${prefix}" />
-<!--eef mounting plate-->
-    <joint name="mounting_plate_joint" type="fixed">
+<!--end effector-->
+    <joint name="${prefix}end_effector_joint" type="fixed">
       <parent link="${prefix}ee_link" />
-      <child link = "mounting_plate" />
-      <origin xyz="0.005 0.0 0.0" rpy="0.0 0.0 0.0" />
-    </joint>
-    <link name="mounting_plate">
-      <visual>
-        <material name="LightGrey">
-          <color rgba="0.752 0.752 0.752 1.0"/>
-        </material>
-  <geometry>
-          <box size="0.01 0.2 0.075"/>
-        </geometry>
-      </visual>
-      <collision>
-        <geometry>
-          <box size="0.01 0.2 0.075"/>
-        </geometry>
-      </collision>
-    </link>
-<!--Forks -->
-   <joint name="fork_left_joint" type="fixed">
-      <parent link="mounting_plate" />
-      <child link = "fork_left" />
-      <origin xyz="0.16 -0.1 0.0" rpy="0.0 0.0 0.0" />
-    </joint>
-    <link name="fork_left">
-      <visual>
-        <material name="LightGrey">
-          <color rgba="0.7 0.7 0.7 1.0"/>
-        </material>
-  <geometry>
-          <box size="0.3 0.01 0.01"/>
-        </geometry>
-      </visual>
-      <collision>
-        <geometry>
-          <box size="0.3 0.01 0.01"/>
-        </geometry>
-      </collision>
-    </link>
-   <joint name="fork_right_joint" type="fixed">
-      <parent link="mounting_plate" />
-      <child link = "fork_right" />
-      <origin xyz="0.16 0.1 0.0" rpy="0.0 0.0 0.0" />
-    </joint>
-    <link name="fork_right">
-      <visual>
-        <material name="LightGrey">
-          <color rgba="0.7 0.7 0.7 1.0"/>
-        </material>
-  <geometry>
-          <box size="0.3 0.01 0.01"/>
-        </geometry>
-      </visual>
-      <collision>
-        <geometry>
-          <box size="0.3 0.01 0.01"/>
-        </geometry>
-      </collision>
-    </link>
-    <!-- Camera -->
-`
-   <joint name="camera_joint" type="fixed">
-      <parent link="mounting_plate" />
-      <child link = "camera" />
-      <origin xyz=" 0.00 0.0 0.065" rpy="-1.57 0.0 -1.57" />
-   </joint>
-  <link name="camera">
-    <!--<collision>
-      <origin xyz="0 0 0" rpy="0 0 1.57"/>
-      <geometry>
-    <box size=" 0.05 0.15 0.05 "/>
-      </geometry>
-    </collision> -->
-    <visual>
-      <origin xyz="0 0 0" rpy="0 0 0"/>
-      <geometry>
-    <box size=" 0.01 0.01 0.01 "/>
-<!--0.05 0.15 0.05 -->
-      </geometry>
-      <material name="red">
-  <color rgba=" 1 0 0 1" />
-      </material>
-    </visual>
-    <inertial>
-      <mass value="0.082" />
-      <origin xyz="0 0 0" rpy="0 0 0"/>
-      <inertia ixx="1e-6" ixy="0" ixz="0" iyy="1e-6" iyz="0" izz="1e-6" />
-    </inertial>
-  </link>
-<joint name="camera_optical_joint" type="fixed">
-    <!-- satisfy both gazebo convention and aruco pkg convetion. looking from x axis and z axis respectively. -->
-    <origin xyz=" 0.0 0.0 0.065" rpy="0 0.0 0" />>
-    <parent link="mounting_plate"/>
-    <child link="camera_link_optical"/>
-  </joint>
- <link name="camera_link_optical">
-  </link>
-<gazebo reference="camera_link_optical">
-    <sensor type="camera" name="camera1">
-      <update_rate>30.0</update_rate>
-      <camera name="camera_head">
-        <horizontal_fov>1.57</horizontal_fov>
-        <image>
-          <width>3840</width>
-          <height>1080</height>
-          <!--<format>R8G8B8</format> -->
-          <format>R8G8B8</format>
-        </image>
-        <clip>
-          <near>0.02</near>
-          <far>300</far>
-        </clip>
-        <noise>
-          <type>gaussian</type>
-          <!-- Noise is sampled independently per pixel on each frame.
-               That pixel's noise value is added to each of its color
-               channels, which at that point lie in the range [0,1]. -->
-          <mean>0.0</mean>
-          <stddev>0.007</stddev>
-        </noise>
-      </camera>
-      <plugin name="camera_controller" filename="libgazebo_ros_camera.so">
-        <alwaysOn>true</alwaysOn>
-        <updateRate>30</updateRate>
-        <cameraName></cameraName>
-        <imageTopicName>/image</imageTopicName>
-        <cameraInfoTopicName>/camera_info</cameraInfoTopicName>
-        <frameName>camera_link</frameName>
-        <hackBaseline>0.07</hackBaseline>
-        <distortionK1>0.0</distortionK1>
-        <distortionK2>0.0</distortionK2>
-        <distortionK3>0.0</distortionK3>
-        <distortionT1>0.0</distortionT1>
-        <distortionT2>0.0</distortionT2>
-      </plugin>
-    </sensor>
-  </gazebo>
-<!--end of camera-->
+      <child link = "${prefix}end_effector_link" />
+      <origin xyz="0.0 0.0 0.0" rpy="0.0 0.0 0.0" />
+    </joint>
+    <link name="${prefix}end_effector_link">
+      <visual>
+        <geometry>
+          <mesh filename="package://ur10_simulation/meshes/visual/end_effector.STL" scale="0.001 0.001 0.001"/>
+        </geometry>
+        <origin xyz="-0.3 0.0 0.0" rpy="${-pi/2} 0.0 ${pi/2}" />
+        <material name="LightGrey">
+          <color rgba="0.7 0.7 0.7 1.0"/>
+        </material>
+      </visual>
+      <xacro:cylinder_inertial radius="0.075" length="0.12" mass="${wrist_3_mass}">
+        <origin xyz="0.0 0.0 0.0" rpy="0 0 0" />
+      </xacro:cylinder_inertial>
+    </link>
+<!--end of end effector-->
     <!-- ROS base_link to UR 'Base' Coordinates transform -->
     <link name="${prefix}base"/>
@@ -438,4 +312,6 @@
       <child link="${prefix}tool0"/>
     </joint>
+    <xacro:ur_arm_transmission prefix="${prefix}" hw_interface="${transmission_hw_interface}" />
+    <xacro:ur_arm_gazebo prefix="${prefix}" />
   </xacro:macro>
 </robot>

Commit message: corrected pose

File: ur10_simulation/urdf/ur10.urdf.xacro (robot description, xacro)
@@ -284,5 +284,5 @@
           <mesh filename="package://ur10_simulation/meshes/visual/end_effector.STL" scale="0.001 0.001 0.001"/>
         </geometry>
-        <origin xyz="-0.3 0.0 0.0" rpy="${-pi/2} 0.0 ${pi/2}" />
+        <origin xyz="0.3 -0.125 0.1" rpy="${-pi/2} 0.0 ${pi/2}" />
         <material name="LightGrey">
           <color rgba="0.7 0.7 0.7 1.0"/>

Commit message: optical joint & end effector added

File: ur10_simulation/urdf/ur10.urdf.xacro (robot description, xacro)
@@ -282,11 +282,17 @@
       <visual>
         <geometry>
-          <mesh filename="package://ur10_simulation/meshes/visual/end_effector.STL" scale="0.001 0.001 0.001"/>
-        </geometry>
-        <origin xyz="0.3 -0.125 0.1" rpy="${-pi/2} 0.0 ${pi/2}" />
-        <material name="LightGrey">
-          <color rgba="0.7 0.7 0.7 1.0"/>
-        </material>
-      </visual>
+          <mesh filename="package://ur10_simulation/meshes/visual/end_effector.STL"/>
+        </geometry>
+        <origin xyz="0.0 0.0 0.0" rpy="${-pi/2} 0.0 ${pi/2}" />
+        <material name="LightGrey">
+          <color rgba="0.7 0.7 0.7 1.0"/>
+        </material>
+      </visual>
+      <collision>
+        <geometry>
+          <mesh filename="package://ur10_simulation/meshes/collision/end_effector.STL"/>
+        </geometry>
+	<origin xyz="0.0 0.0 0.0" rpy="${-pi/2} 0.0 ${pi/2}" />
+      </collision>
       <xacro:cylinder_inertial radius="0.075" length="0.12" mass="${wrist_3_mass}">
         <origin xyz="0.0 0.0 0.0" rpy="0 0 0" />
@@ -294,4 +300,54 @@
     </link>
 <!--end of end effector-->
+<!--camera link-->
+<joint name="camera_optical_joint" type="fixed">
+    <!-- satisfy both gazebo convention and aruco pkg convetion. looking from x axis and z axis respectively. -->
+    <origin xyz=" 0.055 0.06 0.0825" rpy="0 0.0 0" />>
+    <parent link="end_effector_link"/>
+    <child link="camera_link_optical"/>
+  </joint>
+ <link name="camera_link_optical">
+  </link>
+<gazebo reference="camera_link_optical">
+    <sensor type="camera" name="camera1">
+      <update_rate>30.0</update_rate>
+      <camera name="camera_head">
+        <horizontal_fov>1.57</horizontal_fov>
+        <image>
+          <width>3840</width>
+          <height>1080</height>
+          <!--<format>R8G8B8</format> -->
+          <format>R8G8B8</format>
+        </image>
+        <clip>
+          <near>0.02</near>
+          <far>300</far>
+        </clip>
+        <noise>
+          <type>gaussian</type>
+          <!-- Noise is sampled independently per pixel on each frame.
+               That pixel's noise value is added to each of its color
+               channels, which at that point lie in the range [0,1]. -->
+          <mean>0.0</mean>
+          <stddev>0.007</stddev>
+        </noise>
+      </camera>
+      <plugin name="camera_controller" filename="libgazebo_ros_camera.so">
+        <alwaysOn>true</alwaysOn>
+        <updateRate>30</updateRate>
+        <cameraName></cameraName>
+        <imageTopicName>/image</imageTopicName>
+        <cameraInfoTopicName>/camera_info</cameraInfoTopicName>
+        <frameName>camera_link</frameName>
+        <hackBaseline>0.07</hackBaseline>
+        <distortionK1>0.0</distortionK1>
+        <distortionK2>0.0</distortionK2>
+        <distortionK3>0.0</distortionK3>
+        <distortionT1>0.0</distortionT1>
+        <distortionT2>0.0</distortionT2>
+      </plugin>
+    </sensor>
+  </gazebo>
+<!--end of camera link-->
     <!-- ROS base_link to UR 'Base' Coordinates transform -->
     <link name="${prefix}base"/>
